File: protocard/protocard/protocard.kicad_pcb (KiCad board)
At the start: 2 copper layers, 100 x 70 mm, 15 parts, among them J1 SBH11-PBPC-D13-RA-BK, J3 Conn_01x06, J4 Conn_01x06, J5 Conn_01x06, J6 Conn_01x06, U1 74AHC04, U2 4068, U3 PCF8574AP

Commit message: adding assembly, fixes to PCB
Parts:
- removed the J4 at (100.5, 128.5)
- removed J5: Conn_01x06, Connector_PinHeader_2.54mm:PinHeader_1x06_P2.54mm_Vertical
- added J3: Conn_01x06, Connector_PinHeader_2.54mm:PinHeader_1x06_P2.54mm_Vertical, F.Cu at (99.5, 122.8)
- J2: renamed from J3; value Conn_01x06 -> Conn_01x08; footprint Connector_PinHeader_2.54mm:PinHeader_1x06_P2.54mm_Vertical -> Connector_PinHeader_2.54mm:PinHeader_1x08_P2.54mm_Vertical
- J4: renamed from J6; value Conn_01x06 -> Conn_01x03; footprint Connector_PinHeader_2.54mm:PinHeader_1x06_P2.54mm_Vertical -> Connector_PinHeader_2.54mm:PinHeader_1x03_P2.54mm_Vertical
- moved J4 25.9 mm to (99.5, 110.4), turned to 0 degrees
- moved J2 8.36 mm to (99.5, 84.5)
Connections:
- J2 pad 1: Net-(J3-Pin_1) -> A0
- J2 pad 2: Net-(J3-Pin_2) -> A1
- J2 pad 3: Net-(J3-Pin_3) -> Net-(J2-Pin_3)
- J2 pad 4: INP -> Net-(J2-Pin_4)
- J2 pad 5: OUT -> Net-(J2-Pin_5)
- J2 pad 6: WAIT -> INP
- U2 pad 1: Net-(J3-Pin_1) -> Net-(J2-Pin_3)
- U3 pad 14: Net-(J3-Pin_2) -> Net-(J2-Pin_4)
- U3 pad 15: Net-(J3-Pin_3) -> Net-(J2-Pin_5)
Routing:
- net A0: track 0.00 -> 74.0 mm
- net A1: track 0.00 -> 63.2 mm
- net Net-(J3-Pin_2): track 43.9 -> 0.00 mm
- net Net-(J3-Pin_3): track 43.2 -> 0.00 mm
- net Net-(J2-Pin_4): track 0.00 -> 42.6 mm
- net Net-(J3-Pin_1): track 42.5 -> 0.00 mm
- net Net-(J2-Pin_5): track 0.00 -> 41.7 mm
- net Net-(J2-Pin_3): track 0.00 -> 41.2 mm
- net +3V3: track 157.0 -> 125.4 mm, vias 0 -> 2
- net D4: track 54.4 -> 30.6 mm
- net GND: track 21.1 -> 0.00 mm
- net Net-(JP5-C): track 43.1 -> 60.5 mm
- net WAIT: track 75.8 -> 59.1 mm, vias 0 -> 1
- net D3: track 40.4 -> 27.5 mm
- net D5: track 42.0 -> 29.8 mm
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Other:
- board text added: "A0"
- board text added: "A1"
- board text added: "Altair-Duino Prototyping ver 0.95 (C) 2026 M.Brugman"
- board text added: "SET"
- board text added: "UNSET"
- board text removed: "Altair-Duino Prototyping ver 0.9 (C) 2026 M.Brugman"
