File: protocard/protocard/protocard.kicad_sch (KiCad schematic)
At the start: 14 parts, among them J1 SBH11-PBPC-D13-RA-BK, J3 Conn_01x06, J4 Conn_01x06, J5 Conn_01x06, J6 Conn_01x06, U1 74AHC04, U2 4068, U3 PCF8574AP

Commit message: adding assembly, fixes to PCB
Parts:
- removed J5: Conn_01x06, Connector_PinHeader_2.54mm:PinHeader_1x06_P2.54mm_Vertical, symbol Connector_Generic:Conn_01x06
- J2: renamed from J3; value Conn_01x06 -> Conn_01x08; footprint Connector_PinHeader_2.54mm:PinHeader_1x06_P2.54mm_Vertical -> Connector_PinHeader_2.54mm:PinHeader_1x08_P2.54mm_Vertical; symbol Connector_Generic:Conn_01x06 -> Connector_Generic:Conn_01x08
- J4: renamed from J6; value Conn_01x06 -> Conn_01x03; footprint Connector_PinHeader_2.54mm:PinHeader_1x06_P2.54mm_Vertical -> Connector_PinHeader_2.54mm:PinHeader_1x03_P2.54mm_Vertical; symbol Connector_Generic:Conn_01x06 -> Connector_Generic:Conn_01x03
- renumbered J4 to J3
Connections:
- net +3V3: now also J3.1 (Pin_1), J3.2 (Pin_2), J3.3 (Pin_3)
- net +5V: no longer J3.1 (Pin_1), J3.2 (Pin_2), J3.3 (Pin_3)
- net A0: now also J2.1 (Pin_1)
- net A1: now also J2.2 (Pin_2)
- net GND: no longer J4.4 (Pin_4), J4.5 (Pin_5), J4.6 (Pin_6)
- net INP: now also J2.6 (Pin_6); no longer J2.4 (Pin_4)
- net OUT: now also J2.7 (Pin_7); no longer J2.5 (Pin_5)
- net WAIT: now also J2.8 (Pin_8); no longer J2.6 (Pin_6)
- net at U3.14 (SCL): now also J2.4 (Pin_4); no longer J2.2 (Pin_2)
- net at U3.15 (SDA): now also J2.5 (Pin_5); no longer J2.3 (Pin_3)
- net at U2.1 (K): now also J2.3 (Pin_3); no longer J2.1 (Pin_1)
Other:
- note removed: "5V interface header"
